File: esp32_POE.kicad_sch (KiCad schematic)
At the start: 57 parts, among them IC1 TPS2373-4RGWR, J1 Conn_01x03, J10 Conn_01x02, J2 WE-RJ45LAN 10/100BaseT PoE, J3 Conn_01x03, J4 Conn_01x03, J5 Conn_01x03, J8 Conn_01x02, J9 Conn_01x04, SW1 SW_Push, SW2 SW_Push, U1 ESP32-WROOM-32E, U2 XC6206PxxxMR, U5 SN74LVC8T245, U6 LAN8720A

Commit message: Finished setting up the schematic, started basic routing
Parts:
- removed C11: 10uF, Capacitor_THT:CP_Radial_D5.0mm_P2.50mm, symbol Device:C_Polarized
- removed C13: 10uF, Capacitor_SMD:C_0603_1608Metric_Pad1.08x0.95mm_HandSolder, symbol Device:C
- removed C17: 1uF, Capacitor_SMD:C_0603_1608Metric_Pad1.08x0.95mm_HandSolder, symbol Device:C
- removed D2: SMAJ58A, Diode_SMD:D_SMA, symbol Diode:SMAJ58A
- removed D4: 1N4742-12V, Diode_THT:D_DO-41_SOD81_P10.16mm_Horizontal, symbol Diode:1N47xxA
- removed IC1: TPS2373-4RGWR, Package_DFN_QFN:Texas_RGW0020A_VQFN-20-1EP_5x5mm_P0.65mm_EP3.15x3.15mm, symbol TPS2373-4RGWR:TPS2373-4RGWR
- removed J10: Conn_01x02, Connector_PinHeader_2.00mm:PinHeader_1x02_P2.00mm_Vertical, symbol Connector_Generic:Conn_01x02
- removed J2: WE-RJ45LAN 10/100BaseT PoE, custom:7499211125, symbol Custom:WE-RJ45LAN 10/100BaseT PoE
- removed J8: Conn_01x02, TerminalBlock_MetzConnect:TerminalBlock_MetzConnect_Type055_RT01502HDWU_1x02_P5.00mm_Horizontal, symbol Connector_Generic:Conn_01x02
- removed R35, R36: 100k, Resistor_SMD:R_0603_1608Metric_Pad0.98x0.95mm_HandSolder, symbol Device:R
- removed R37: 1.3k, Resistor_THT:R_Axial_DIN0207_L6.3mm_D2.5mm_P10.16mm_Horizontal, symbol Device:R
- removed U3: ~, custom:Mini_DC-DC_Buck, symbol Custom:Mini_DC-DC_Buck
- added C1: 10uF, Capacitor_SMD:C_0603_1608Metric, symbol Device:C
- added C12, C14: 22uF/35V, Capacitor_SMD:C_0805_2012Metric, symbol Device:C
- added C3, C5: 4.7uF,100V, Capacitor_SMD:C_1206_3216Metric, symbol Device:C
- added C4: .1uF, Capacitor_SMD:C_0603_1608Metric, symbol Device:C
- added C7: 56pF, Capacitor_SMD:C_0603_1608Metric, symbol Device:C
- added C9: .1uF,10V, Capacitor_SMD:C_0603_1608Metric, symbol Device:C
- added D1, D4, D6, D7: LED, LED_SMD:LED_0603_1608Metric, symbol Device:LED
- added D2, D5: SDT20B100D1-13, Package_TO_SOT_SMD:TO-252-2, symbol Device:D_Schottky
- added D3: 51V, Diode_SMD:D_SMA, symbol Device:D_Zener
- added J1: Barrel_Jack_Switch, Connector_BarrelJack:BarrelJack_Horizontal, symbol Connector:Barrel_Jack_Switch
- added J2: Conn_02x03_Odd_Even, Connector_PinHeader_2.54mm:PinHeader_2x03_P2.54mm_Vertical, symbol Connector_Generic:Conn_02x03_Odd_Even
- added J4: Conn_01x04, Connector_PinSocket_1.27mm:PinSocket_1x04_P1.27mm_Vertical, symbol Connector_Generic:Conn_01x04
- added L1: SMMS1770-330M, Inductor_SMD:L_Vishay_IHLP-6767, symbol Device:L
- added R1, R25, R9: 3k, Resistor_SMD:R_0603_1608Metric, symbol Device:R
- added R10: 63.4, Resistor_SMD:R_0603_1608Metric, symbol Device:R
- added R11: 90.9, Resistor_SMD:R_0603_1608Metric, symbol Device:R
- added R12: 49.9k, Resistor_SMD:R_0603_1608Metric, symbol Device:R
- added R21: 53.6k, Resistor_SMD:R_0603_1608Metric, symbol Device:R
- added R22: 10.2k, Resistor_SMD:R_0603_1608Metric, symbol Device:R
- added R23: 143k, Resistor_SMD:R_0603_1608Metric, symbol Device:R
- added R24: 294k, Resistor_SMD:R_0603_1608Metric, symbol Device:R
- added R27, R28: 10, Resistor_SMD:R_0603_1608Metric, symbol Device:R
- added R3: 118k, Resistor_SMD:R_0603_1608Metric, symbol Device:R
- added R4: 36.5k, Resistor_SMD:R_0603_1608Metric, symbol Device:R
- added R6: 25k, Resistor_SMD:R_0603_1608Metric, symbol Device:R
- added R7: 13.3k, Resistor_SMD:R_0603_1608Metric, symbol Device:R
- added R8: 220k, Resistor_SMD:R_0603_1608Metric, symbol Device:R
- added U1: HY931147C, HY931147C:HY931147C, symbol HY931147C:HY931147C
- added U2: TPS2372, Package_DFN_QFN:Texas_RGW0020A_VQFN-20-1EP_5x5mm_P0.65mm_EP3.15x3.15mm, symbol Custom:TPS2372
- added U3: TPS54560BDDA, Package_SO:Texas_R-PDSO-G8_EP2.95x4.9mm_Mask2.4x3.1mm_ThermalVias, symbol Regulator_Switching:TPS54560BDDA
- C10: renamed from C18; footprint Capacitor_SMD:C_0603_1608Metric_Pad1.08x0.95mm_HandSolder -> Capacitor_SMD:C_0603_1608Metric
- C11: renamed from C15; footprint Capacitor_SMD:C_0603_1608Metric_Pad1.08x0.95mm_HandSolder -> Capacitor_SMD:C_0603_1608Metric
- C13: renamed from C19; footprint Capacitor_SMD:C_0603_1608Metric_Pad1.08x0.95mm_HandSolder -> Capacitor_SMD:C_0603_1608Metric
- C15: renamed from C20; footprint Capacitor_SMD:C_0603_1608Metric_Pad1.08x0.95mm_HandSolder -> Capacitor_SMD:C_0603_1608Metric
- C16: value .1uF -> 22uF/35V; footprint Capacitor_SMD:C_0603_1608Metric_Pad1.08x0.95mm_HandSolder -> Capacitor_SMD:C_0805_2012Metric
- C17: renamed from C3; footprint Capacitor_SMD:C_0603_1608Metric_Pad1.08x0.95mm_HandSolder -> Capacitor_SMD:C_0603_1608Metric
- C18: renamed from C4; footprint Capacitor_SMD:C_0603_1608Metric_Pad1.08x0.95mm_HandSolder -> Capacitor_SMD:C_0603_1608Metric
- C19: renamed from C5; footprint Capacitor_SMD:C_0603_1608Metric_Pad1.08x0.95mm_HandSolder -> Capacitor_SMD:C_0603_1608Metric
- C2: renamed from C14; footprint Capacitor_SMD:C_0603_1608Metric_Pad1.08x0.95mm_HandSolder -> Capacitor_SMD:C_0603_1608Metric
- C20: renamed from C6; footprint Capacitor_SMD:C_0603_1608Metric_Pad1.08x0.95mm_HandSolder -> Capacitor_SMD:C_0603_1608Metric
- C21: renamed from C2; footprint Capacitor_SMD:C_0603_1608Metric_Pad1.08x0.95mm_HandSolder -> Capacitor_SMD:C_0603_1608Metric
- C22: renamed from C1; footprint Capacitor_SMD:C_0603_1608Metric_Pad1.08x0.95mm_HandSolder -> Capacitor_SMD:C_0603_1608Metric
- C6: renamed from C7; footprint Capacitor_SMD:C_0603_1608Metric_Pad1.08x0.95mm_HandSolder -> Capacitor_SMD:C_0603_1608Metric
- C8: value .1uF -> 1200pF; footprint Capacitor_SMD:C_0603_1608Metric_Pad1.08x0.95mm_HandSolder -> Capacitor_SMD:C_0603_1608Metric
- J5: footprint (none) -> Connector_JST:JST_XH_B3B-XH-AM_1x03_P2.50mm_Vertical
- J6: renamed from J4; footprint (none) -> Connector_JST:JST_XH_B3B-XH-AM_1x03_P2.50mm_Vertical
- J7: renamed from J3; footprint (none) -> Connector_JST:JST_XH_B3B-XH-AM_1x03_P2.50mm_Vertical
- J8: renamed from J1; footprint (none) -> Connector_JST:JST_XH_B3B-XH-AM_1x03_P2.50mm_Vertical
- R18: renamed from R25; footprint Resistor_SMD:R_0603_1608Metric_Pad0.98x0.95mm_HandSolder -> Resistor_SMD:R_0603_1608Metric
- R19: renamed from R7; footprint Resistor_SMD:R_0603_1608Metric_Pad0.98x0.95mm_HandSolder -> Resistor_SMD:R_0603_1608Metric
- R2: renamed from R5; footprint Resistor_SMD:R_0603_1608Metric_Pad0.98x0.95mm_HandSolder -> Resistor_SMD:R_0603_1608Metric
- R20: renamed from R6; footprint Resistor_SMD:R_0603_1608Metric_Pad0.98x0.95mm_HandSolder -> Resistor_SMD:R_0603_1608Metric
- R26: value 100 -> 10; footprint Resistor_SMD:R_0603_1608Metric_Pad0.98x0.95mm_HandSolder -> Resistor_SMD:R_0603_1608Metric
- R29: value 18k -> 10; footprint Resistor_SMD:R_0603_1608Metric_Pad0.98x0.95mm_HandSolder -> Resistor_SMD:R_0603_1608Metric
- R30: value 7.5k -> 10; footprint Resistor_SMD:R_0603_1608Metric_Pad0.98x0.95mm_HandSolder -> Resistor_SMD:R_0603_1608Metric
- R31: value 62 -> 10; footprint Resistor_SMD:R_0603_1608Metric_Pad0.98x0.95mm_HandSolder -> Resistor_SMD:R_0603_1608Metric
- R32: value 1k -> 10; footprint Resistor_SMD:R_0603_1608Metric_Pad0.98x0.95mm_HandSolder -> Resistor_SMD:R_0603_1608Metric
- R33: value 1 -> 10; footprint Resistor_SMD:R_0603_1608Metric_Pad0.98x0.95mm_HandSolder -> Resistor_SMD:R_0603_1608Metric
- R34: footprint Resistor_SMD:R_0603_1608Metric_Pad0.98x0.95mm_HandSolder -> Resistor_SMD:R_0603_1608Metric
- R35: renamed from R2; footprint Resistor_SMD:R_0603_1608Metric_Pad0.98x0.95mm_HandSolder -> Resistor_SMD:R_0603_1608Metric
- R36: renamed from R1; footprint Resistor_SMD:R_0603_1608Metric_Pad0.98x0.95mm_HandSolder -> Resistor_SMD:R_0603_1608Metric
- R5: renamed from R24; footprint Resistor_SMD:R_0603_1608Metric_Pad0.98x0.95mm_HandSolder -> Resistor_SMD:R_0603_1608Metric
- SW1, SW2: footprint Button_Switch_THT:SW_PUSH_6mm_H4.3mm -> Button_Switch_SMD:SW_Push_SPST_NO_Alps_SKRK; LCSC (none) -> C720477
- renumbered J9 to J3, R3 to R13, R4 to R14, R22 to R15, R23 to R16, R21 to R17, U6 to U4, U1 to U6, U2 to U7
Connections:
- net +3.3V: now also R5.1, C1.2, D7.2 (A), U1.P$13 (G+), U1.P$3 (RXCT), U1.P$4 (TXCT); no longer R5.2
- net +5V: no longer C19.1, U7.3 (VI)
- net CHANNEL1: now also U5.14 (B8); no longer U5.17 (B5)
- net CHANNEL2: now also U5.15 (B7); no longer U5.16 (B6)
- net CHANNEL3: now also U5.16 (B6); no longer U5.15 (B7)
- net CHANNEL4: now also U5.17 (B5); no longer U5.14 (B8)
- net ETH_MDIO: now also R5.2; no longer R5.1
- net ETH_RST: now also U6.24 (IO2)
- net GND: now also C8.1, J5.1 (Pin_1), J6.1 (Pin_1), J7.1 (Pin_1), J8.1 (Pin_1), R18.1, R34.1, C1.1, C12.2, C14.2, C3.2, C5.2, C7.1, D5.1 (A), D5.3 (A), J1.2, J1.3, J4.1 (Pin_1), R1.1, R22.1, R25.1, R4.1, R8.2, U1.GND1, U1.GND2, U1.P$12 (Y-), U2.11 (RTN), U2.12 (RTN), U3.7 (GND), U3.9 (GND); no longer J5.3 (Pin_3), J6.3 (Pin_3), J7.3 (Pin_3), J8.3 (Pin_3), R26.1
- net RX: now also J4.2 (Pin_2)
- net TX: now also J4.3 (Pin_3)
- net at J3.1 (Pin_1): now also R26.2; no longer U5.3 (A1)
- net at J3.2 (Pin_2): now also R27.2; no longer U5.4 (A2)
- net at J3.3 (Pin_3): now also R28.2; no longer U5.5 (A3)
- net at J3.4 (Pin_4): now also R29.2; no longer U5.6 (A4)
- net VCC: now reaches C16.1
- net VCC: now also C19.1, J5.3 (Pin_3), J6.3 (Pin_3), J7.3 (Pin_3), J8.3 (Pin_3), U7.3 (VI), C12.1, C14.1, D6.2 (A), J4.4 (Pin_4), L1.2, R21.2, R23.2, R24.2
- net at J5.2 (Pin_2): now also R30.2; no longer U5.7 (A5)
- net 5V_CHANNEL4: now reaches R30.1
- net 5V_CHANNEL4: now also U5.7 (A5)
- net 5V_CHANNEL5: now reaches R29.1
- net 5V_CHANNEL5: now also U5.6 (A4); no longer R30.2
- net at J7.2 (Pin_2): now also R32.2; no longer U5.9 (A7)
- net at J8.2 (Pin_2): now also R33.2; no longer U5.10 (A8)
- net at J6.2 (Pin_2): now also R31.2; no longer U5.8 (A6)
- net 5V_CHANNEL1: now reaches R33.1
- net 5V_CHANNEL1: now also U5.10 (A8)
- net 5V_CHANNEL2: now reaches R32.1
- net 5V_CHANNEL2: now also U5.9 (A7); no longer R34.1
- net BRKOUT1 renamed CHANNEL5
- net BRKOUT2 renamed CHANNEL6
- net BRKOUT3 renamed CHANNEL7
- net BRKOUT4 renamed CHANNEL8
- net LED1 renamed LED1/REGOFF
- net LED1/REGOFF: now also U1.P$11 (Y+)
- net LED2 renamed LED2/nINTSEL
- net LED2/nINTSEL: now also U1.P$14 (G-)
- net RD+ renamed RX+
- net RX+: now also U1.P$6 (TX-)
- net RD- renamed RX-
- net RX-: now also U1.P$5 (TX+)
- net TD+ renamed TX+
- net TX+: now also U1.P$2 (RX-)
- net TD- renamed TX-
- net TX-: now also U1.P$1 (RX+)
- removed net V+: C8.1, J5.1 (Pin_1), J6.1 (Pin_1), J7.1 (Pin_1), J8.1 (Pin_1), R29.2
- removed net V-: C8.2, R31.1, R32.2, R34.2
- new net: D7.1 (K), R34.2
- new net: D1.1 (K), R1.2
- new net: C8.2, R7.2
- new net: D6.1 (K), R25.2
- new net: R6.2, U2.2 (DEN)
- new net: J2.4 (Pin_4), R23.1
- new net: R10.2, U2.3 (CLSA)
- new net: D1.2 (A), D2.1 (A), D2.3 (A), J1.1
- new net: J2.2 (Pin_2), R21.1
- new net: R3.1, R4.2, U3.3 (EN)
- new net: C9.2, U3.1 (BOOT)
- new net: R8.1, U3.4 (RT/CLK)
- new net: C7.2, R7.1, U3.6 (COMP)
- new net: C9.1, D5.2 (K), L1.1, U3.8 (SW)
- new net: J2.6 (Pin_6), R24.1
- new net: R9.1, U2.18 (TPH)
- new net: D4.1 (K), R9.2
- new net: U2.14 (NC), U2.15 (NC), U2.20 (NC)
- new net: R11.1, U2.6 (CLSB)
- new net: R12.1, U2.7 (REF)
- new net 5V_CHANNEL3: R31.1, U5.8 (A6)
- new net 5V_CHANNEL6: R28.1, U5.5 (A3)
- new net 5V_CHANNEL7: R27.1, U5.4 (A2)
- new net 5V_CHANNEL8: R26.1, U5.3 (A1)
- new net FB: J2.1 (Pin_1), J2.3 (Pin_3), J2.5 (Pin_5), R22.2, U3.5 (FB)
- new net POE_V+: C3.1, C4.1, C5.1, D2.2 (K), D3.1 (K), D4.2 (A), R3.2, R6.1, U1.P$9 (V+), U2.1 (VDD), U3.2 (VIN)
- new net POE_V-: C4.2, D3.2 (A), R10.1, R11.2, R12.2, U1.P$10 (V-), U2.21 (EPAD), U2.4 (VSS), U2.5 (VSS)
- no-connect marks 12 -> 14
Other:
- note added: "20A, 100V 9.2W dissipated =22 deg temp rise"
- note added: "40 uF derated"
- note added: "440kHz"
- note added: "CLSA = 63.4, CLSB = 90.0 => PD Class 8, 71W"
- note added: "ESP32-WLED-PoE"
- note added: "Iripple = 1.65A IL(rms) = 6A IL(max) = 6.83A"
- note added: "Made by Whitebow"
- note added: "Min. inductor : 5.9 uH for 5V output 11.9uH for 12V output 32 uH for 24V output"
- note added: "Summoned these values out of my ass"
- note added: "Swapped + and - for wayyy easier routing Auto-MDIX should work ?"
- note added: "TOTAL POWER DISSIPATED = 1.67W DeltaT = 70 degC, consider radiator"
- note added: "UVLO @ 4.5V START @ 4.9V"
- note added: "Vin(max) = 48V Iout(max) = 9A@5V, 6A@12V, 3A@24V Vout = 5V, 12V or 24V"
- note added: "Vout = 5V @ 53.6k = 12V @ 143k = 23.85V @ 294k"
- note added: "WS2811 specifies 1V ripple max. When switching 9A@5V, Cout > 40 uF Icout(rms) = .25A"
- note added: "XR1770-330M also works"
- note added: "v4.0"
- note removed: "23.7k < R_DEN < 26.3k"
- note removed: "R_CLSA = 63.4"
- note removed: "R_CLSB = 90.9"
- moved on the sheet: C10, C11, C13, C15, C17, C18, C19, C2, C20, C21, C22, C6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

Commit message: Finished 1st routing pass, reduced size of PCB
Parts:
- R26, R27, R28, R29, R30, R31, R32, R33: value 10 -> 120
Connections:
- net +3.3V: now also J4.4 (Pin_4)
- net CHANNEL1: now also U6.29 (IO5); no longer U6.26 (IO4)
- net CHANNEL2: now also U6.27 (IO16); no longer U6.29 (IO5)
- net CHANNEL3: now also U6.26 (IO4); no longer U6.14 (IO12)
- net CHANNEL4: now also U6.23 (IO15); no longer U6.13 (IO14)
- net CHANNEL5: now also U6.8 (IO32); no longer U6.23 (IO15)
- net CHANNEL6: now also U6.9 (IO33); no longer U6.27 (IO16)
- net CHANNEL7: now also U6.14 (IO12); no longer U6.8 (IO32)
- net CHANNEL8: now also U6.13 (IO14); no longer U6.9 (IO33)
- net VCC: no longer J4.4 (Pin_4)
Changed lines of the file:
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@@
 		)
 	)
-	(wire
-		(pts
-			(xy 303.53 95.25) (xy 317.5 95.25)
-		)
-		(stroke
-			(width 0)
-			(type default)
-			(color 194 0 194 1)
-		)
-	)
 	(bus
 		(pts
@@
 	(wire
 		(pts
+			(xy 303.53 95.25) (xy 317.5 95.25)
+		)
+		(stroke
+			(width 0)
+			(type default)
+			(color 194 0 194 1)
+		)
+	)
+	(wire
+		(pts
 			(xy 359.41 238.76) (xy 359.41 237.49)
 		)
@@
 	(wire
 		(pts
-			(xy 303.53 97.79) (xy 317.5 97.79)
-		)
-		(stroke
-			(width 0)
-			(type default)
-			(color 194 0 194 1)
-		)
-	)
-	(wire
-		(pts
 			(xy 374.65 167.64) (xy 375.92 167.64)
 		)
@@
 	(wire
 		(pts
+			(xy 303.53 97.79) (xy 317.5 97.79)
+		)
+		(stroke
+			(width 0)
+			(type default)
+			(color 194 0 194 1)
+		)
+	)
+	(wire
+		(pts
 			(xy 67.31 115.57) (xy 68.58 115.57)
 		)
@@
 		)
 	)
+	(label "CHANNEL2"
+		(at 303.53 69.85 0)
+		(effects
+			(font
+				(size 1.27 1.27)
+				(color 72 0 72 1)
+			)
+			(justify left bottom)
+		)
+	)
 	(label "ETH_RST"
 		(at 154.94 86.36 0)
@@
 		)
 	)
+	(label "CHANNEL4"
+		(at 303.53 67.31 0)
+		(effects
+			(font
+				(size 1.27 1.27)
+				(color 72 0 72 1)
+			)
+			(justify left bottom)
+		)
+	)
 	(label "5V_CHANNEL2"
 		(at 336.55 179.07 0)
@@
 		)
 	)
-	(label "CHANNEL1"
-		(at 303.53 54.61 0)
-		(effects
-			(font
-				(size 1.27 1.27)
-				(color 72 0 72 1)
-			)
-			(justify left bottom)
-		)
-	)
 	(label "ETH_RXD1"
 		(at 303.53 90.17 0)
@@
 		)
 	)
-	(label "CHANNEL6"
-		(at 303.53 69.85 0)
-		(effects
-			(font
-				(size 1.27 1.27)
-				(color 72 0 72 1)
-			)
-			(justify left bottom)
-		)
-	)
 	(label "CHANNEL5"
 		(at 303.53 163.83 0)
@@
 		)
 	)
+	(label "CHANNEL3"
+		(at 303.53 54.61 0)
+		(effects
+			(font
+				(size 1.27 1.27)
+				(color 72 0 72 1)
+			)
+			(justify left bottom)
+		)
+	)
+	(label "CHANNEL7"
+		(at 303.53 59.69 0)
+		(effects
+			(font
+				(size 1.27 1.27)
+				(color 72 0 72 1)
+			)
+			(justify left bottom)
+		)
+	)
 	(label "ETH_RXD0"
 		(at 172.72 66.04 0)
@@
 		)
 	)
-	(label "CHANNEL3"
-		(at 303.53 59.69 0)
-		(effects
-			(font
-				(size 1.27 1.27)
-				(color 72 0 72 1)
-			)
-			(justify left bottom)
-		)
-	)
 	(label "POE_V+"
 		(at 93.98 110.49 0)
@@
 		)
 	)
-	(label "CHANNEL4"
+	(label "CHANNEL8"
 		(at 303.53 64.77 0)
 		(effects
@@
 		)
 	)
+	(label "CHANNEL5"
+		(at 303.53 95.25 0)
+		(effects
+			(font
+				(size 1.27 1.27)
+				(color 72 0 72 1)
+			)
+			(justify left bottom)
+		)
+	)
+	(label "CHANNEL1"
+		(at 303.53 57.15 0)
+		(effects
+			(font
+				(size 1.27 1.27)
+				(color 72 0 72 1)
+			)
+			(justify left bottom)
+		)
+	)
 	(label "TX-"
 		(at 275.59 66.04 0)
@@
 		)
 	)
-	(label "CHANNEL7"
-		(at 304.8 95.25 0)
+	(label "CHANNEL6"
+		(at 303.53 97.79 0)
 		(effects
 			(font
@@
 		)
 	)
-	(label "CHANNEL2"
-		(at 303.53 57.15 0)
-		(effects
-			(font
-				(size 1.27 1.27)
-				(color 72 0 72 1)
-			)
-			(justify left bottom)
-		)
-	)
 	(label "POE_V+"
 		(at 116.84 224.79 0)
@@
 		)
 	)
-	(label "CHANNEL5"
-		(at 303.53 67.31 0)
-		(effects
-			(font
-				(size 1.27 1.27)
-				(color 72 0 72 1)
-			)
-			(justify left bottom)
-		)
-	)
 	(label "CHANNEL2"
 		(at 303.53 179.07 0)
@@
 		)
 	)
-	(label "CHANNEL8"
-		(at 304.8 97.79 0)
-		(effects
-			(font
-				(size 1.27 1.27)
-				(color 72 0 72 1)
-			)
-			(justify left bottom)
-		)
-	)
 	(label "ETH_CLK"
 		(at 179.07 93.98 0)
@@
 	)
 	(symbol
-		(lib_id "power:VCC")
-		(at 386.08 99.06 0)
-		(mirror y)
-		(unit 1)
-		(exclude_from_sim no)
-		(in_bom yes)
-		(on_board yes)
-		(dnp no)
-		(property "Reference" "#PWR048"
-			(at 386.08 102.87 0)
-			(effects
-				(font
-					(size 1.27 1.27)
-				)
-				(hide yes)
-			)
-		)
-		(property "Value" "VCC"
-			(at 389.128 97.79 0)
-			(effects
-				(font
-					(size 1.27 1.27)
-				)
-			)
-		)
-		(property "Footprint" ""
-			(at 386.08 99.06 0)
-			(effects
-				(font
-					(size 1.27 1.27)
-				)
-				(hide yes)
-			)
-		)
-		(property "Datasheet" ""
-			(at 386.08 99.06 0)
-			(effects
-				(font
-					(size 1.27 1.27)
-				)
-				(hide yes)
-			)
-		)
-		(property "Description" "Power symbol creates a global label with name \"VCC\""
-			(at 386.08 99.06 0)
-			(effects
-				(font
-					(size 1.27 1.27)
-				)
-				(hide yes)
-			)
-		)
-		(pin "1"
-		)
-		(instances
-			(project "esp32_POE"
-				(path "/2d9203e9-fefd-4c2a-a523-572538ad59ab"
-					(reference "#PWR048")
-					(unit 1)
-				)
-			)
-		)
-	)
-	(symbol
 		(lib_id "HY931147C:HY931147C")
 		(at 54.61 49.53 0)
@@
 			)
 		)
-		(property "Value" "10"
+		(property "Value" "120"
 			(at 358.14 163.83 90)
 			(effects
@@
 			)
 		)
-		(property "Value" "10"
+		(property "Value" "120"
 			(at 358.14 158.75 90)
 			(effects
@@
 			)
 		)
-		(property "Value" "10"
+		(property "Value" "120"
 			(at 358.14 153.67 90)
 			(effects
@@
 			)
 		)
-		(property "Value" "10"
+		(property "Value" "120"
 			(at 379.73 176.53 90)
 			(effects
@@
 			)
 		)
-		(property "Value" "10"
+		(property "Value" "120"
 			(at 379.73 167.64 90)
 			(effects
@@
 			)
 		)
-		(property "Value" "10"
+		(property "Value" "120"
 			(at 358.14 148.59 90)
 			(effects
@@
 	)
 	(symbol
+		(lib_id "power:+3.3V")
+		(at 386.08 99.06 0)
+		(unit 1)
+		(exclude_from_sim no)
+		(in_bom yes)
+		(on_board yes)
+		(dnp no)
+		(fields_autoplaced yes)
+		(property "Reference" "#PWR048"
+			(at 386.08 102.87 0)
+			(effects
+				(font
+					(size 1.27 1.27)
+				)
+				(hide yes)
+			)
+		)
+		(property "Value" "+3.3V"
+			(at 386.08 93.98 0)
+			(effects
+				(font
+					(size 1.27 1.27)
+				)
+			)
+		)
+		(property "Footprint" ""
+			(at 386.08 99.06 0)
+			(effects
+				(font
+					(size 1.27 1.27)
+				)
+				(hide yes)
+			)
+		)
+		(property "Datasheet" ""
+			(at 386.08 99.06 0)
+			(effects
+				(font
+					(size 1.27 1.27)
+				)
+				(hide yes)
+			)
+		)
+		(property "Description" "Power symbol creates a global label with name \"+3.3V\""
+			(at 386.08 99.06 0)
+			(effects
+				(font
+					(size 1.27 1.27)
+				)
+				(hide yes)
+			)
+		)
+		(pin "1"
+		)
+		(instances
+			(project "esp32_POE"
+				(path "/2d9203e9-fefd-4c2a-a523-572538ad59ab"
+					(reference "#PWR048")
+					(unit 1)
+				)
+			)
+		)
+	)
+	(symbol
 		(lib_id "Device:C")
 		(at 346.71 234.95 0)
@@
 			)
 		)
-		(property "Value" "10"
+		(property "Value" "120"
 			(at 379.984 185.42 90)
 			(effects
@@
 			)
 		)
-		(property "Value" "10"
+		(property "Value" "120"
 			(at 378.46 158.75 90)
 			(effects
